File: hs-64-spi.brd (EAGLE design)
At the start: 37.5 x 18.8 mm, 25 parts, among them J1 DF40C-70DP-0.4V(51), J2 A79622-001, U1 RHD2064_BGA, U2 ADXL335_IDAX

Commit message: Corrected C7 value to 4.7uF.
Parts:
- C7: value 1u -> 4.7u
Changed lines of the file:
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@@
 <attribute name="NAME" x="-4.617125" y="2.162" size="0.8128" layer="25" font="vector" ratio="19"/>
 </element>
-<element name="C7" library="jonnew" package="0402" value="1u" x="-2.9816" y="-0.008" smashed="yes" rot="R90">
+<element name="C7" library="jonnew" package="0402" value="4.7u" x="-2.9816" y="-0.008" smashed="yes" rot="R90">
 <attribute name="NAME" x="-3.6784" y="-2.0618" size="0.8128" layer="25" font="vector" ratio="19"/>
 </element>

Commit message: Updated Hirose (J1) schematic.
Connections:
- removed net ISTIM: J1.1
- removed net LED-1: J1.34
- removed net LED-2: J1.35
Changed lines of the file:
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@@
 </elements>
 <signals>
-<signal name="LED-2">
-<contactref element="J1" pad="35"/>
-</signal>
 <signal name="VCOAX">
 <contactref element="J1" pad="36"/>
@@
 <contactref element="U1" pad="A9"/>
 <wire x1="0" y1="-0.585" x2="0" y2="-2" width="0.09" layer="16"/>
-</signal>
-<signal name="LED-1">
-<contactref element="J1" pad="34"/>
 </signal>
 <signal name="REF">
@@
 <wire x1="-6.3824" y1="-4.7116" x2="-6.9216" y2="-4.1724" width="0.09" layer="16"/>
 </signal>
-<signal name="ISTIM">
-<contactref element="J1" pad="1"/>
-</signal>
 <signal name="RESV(VCCIO)">
